File: MQXX Gas Sensor V1.0/MQxx Gas Sensor V1.0/MQxx Gas Sensor V1.0.sch (KiCad schematic (older format))
At the start: 7 parts, among them J1 Conn_01x03_Male, J2 1935161, J3 1935161, Q1 IRF520PBF

Commit message: MQxx Gas Sensor V1.0
Parts:
- removed J1: Conn_01x03_Male, Connector_PinHeader_2.54mm:PinHeader_1x03_P2.54mm_Horizontal, symbol Connector:Conn_01x03_Male
- removed J2, J3: 1935161, TerminalBlock:TerminalBlock_Altech_AK300-2_P5.00mm, symbol dk_Terminal-Blocks-Wire-to-Board:1935161
- removed Q1: IRF520PBF, digikey-footprints:TO-220-3, symbol dk_Transistors-FETs-MOSFETs-Single:IRF520PBF
- added C1, C2: 0.1uF, Capacitor_SMD:C_0805_2012Metric_Pad1.15x1.40mm_HandSolder, symbol Device:C
- added D2: DO_LED, LED_SMD:LED_0805_2012Metric_Pad1.15x1.40mm_HandSolder, symbol Device:LED
- added J1: Conn_01x04_Male, Connector_PinHeader_2.54mm:PinHeader_1x04_P2.54mm_Vertical, symbol Connector:Conn_01x04_Male
- added R3: 5.1E, Resistor_SMD:R_0805_2012Metric_Pad1.15x1.40mm_HandSolder, symbol Device:R
- added R4: 4.7K, Resistor_SMD:R_0805_2012Metric_Pad1.15x1.40mm_HandSolder, symbol Device:R
- added RV1: 10K, Potentiometer_THT:Potentiometer_Vishay_T73YP_Vertical, symbol Device:R_POT
- added U1: LM393, Package_SO:SOIC-8-1EP_3.9x4.9mm_P1.27mm_EP2.29x3mm, symbol Device:Opamp_Dual_Generic
- added U?1: MQ-X, Sensor:MQ-6, symbol Sensor_Gas:MQ-6
- D1: value RED -> PWR_LED
Connections:
- net labels added: +5V, AOUT, DOUT
- net labels removed: SIG, V+, V-, VIN
- wire segments 25 -> 46
- no-connect marks 1 -> 0
